Commit message: Brazo de Milo: cinemática inversa con lift, control en Gazebo y marcador en RViz
- andesrobot_description: articulaciones del brazo revolute con límites provisorios (±π),
  frame gripper_tcp (punto de agarre medido en las mallas de los dedos), argumento
  arm_control que agrega ros2_control del brazo/lift/pinza en Gazebo
  (andesrobot.arm_control.xacro).
- andesrobot_arm (nuevo): cinemática directa/inversa leída del URDF (DLS ponderado,
  7 articulaciones con el lift), arm_ik_node, arm_marker_node, controladores,
  arm_sim.launch.py, RViz, tests y docs/BRAZO.md.
- ./sim.sh brazo, gazebo-ros2-control en el Dockerfile, README y ROBOT.md.

Co-Authored-By: Claude Opus 5.5 <noreply@anthropic.com>

File: ros2_ws/src/andesrobot_description/urdf/andesrobot.urdf.xacro (robot description, xacro)
@@ -41,5 +41,5 @@
 <xacro:property name="lock_arm" value="${'$(arg lock_arm)' == 'true'}"/>
 <!-- Tipo de articulación del brazo: fixed si lock_arm, si no continuous (gira) / prismatic (desliza). -->
-<xacro:property name="arm_joint_type" value="${'fixed' if lock_arm else 'continuous'}"/>
+<xacro:property name="arm_joint_type" value="${'fixed' if lock_arm else 'revolute'}"/>
 <xacro:property name="prismatic_joint_type" value="${'fixed' if lock_arm else 'prismatic'}"/>
 <!-- simple_collision:=true -> la física usa cajas/cilindros en vez de las mallas CAD (estable y rápido en Gazebo).
@@ -47,4 +47,10 @@
 <xacro:arg name="simple_collision" default="false"/>
 <xacro:property name="simple_collision" value="${'$(arg simple_collision)' == 'true'}"/>
+<!-- arm_control:=true -> el brazo, el lift y la pinza se mueven con ros2_control dentro de Gazebo
+     (andesrobot.arm_control.xacro). Lo usa andesrobot_arm/arm_sim.launch.py. Requiere lock_arm:=false.
+     arm_controllers_file = YAML de los controladores que carga el plugin gazebo_ros2_control. -->
+<xacro:arg name="arm_control" default="false"/>
+<xacro:property name="arm_control" value="${'$(arg arm_control)' == 'true'}"/>
+<xacro:arg name="arm_controllers_file" default=""/>
 <!-- Interruptores de sensores simulados (para depurar). Los usa andesrobot.sim.xacro. -->
 <xacro:arg name="sim_lidar" default="true"/>
@@ -499,7 +505,18 @@
 </link>
 <!-- ================================== ARTICULACIONES (joints) ==================================
-     Las articulaciones del brazo quedan "continuous" (sin topes) SOLO hasta medir los topes físicos.
-     Antes de mover el brazo real (o usar MoveIt), cambiar a "revolute" con límites medidos
-     (lower/upper en rad, velocity, effort). Con lock_arm:=true son "fixed". -->
+     Las articulaciones del brazo son "revolute" con límites PROVISORIOS: ±π (una vuelta completa,
+     o sea sin restringir el rango), 20 N·m y 1 rad/s. Sirven para simular y para la cinemática
+     inversa, pero NO son los topes reales: antes de mover el brazo real (o usar MoveIt), medir los
+     topes físicos y los motores y cambiar estas 4 propiedades. Con lock_arm:=true son "fixed". -->
+<xacro:property name="arm_lower" value="${-pi}"/>
+<xacro:property name="arm_upper" value="${pi}"/>
+<xacro:property name="arm_effort" value="20.0"/>
+<xacro:property name="arm_velocity" value="1.0"/>
+<!-- Límite de cada articulación del brazo (las "fixed" no llevan límite). -->
+<xacro:macro name="arm_limit">
+  <xacro:unless value="${lock_arm}">
+    <limit lower="${arm_lower}" upper="${arm_upper}" effort="${arm_effort}" velocity="${arm_velocity}"/>
+  </xacro:unless>
+</xacro:macro>
 <!-- Brazo 1: gira la base del brazo alrededor de Z (vertical). -->
 <joint name="joint_1" type="${arm_joint_type}">
@@ -512,4 +529,5 @@
   <!-- Amortiguación y roce de la articulación (solo para la simulación). -->
   <dynamics damping="0.08" friction="0.02"/>
+  <xacro:arm_limit/>
 </joint>
 <!-- Brazo 2 (hombro): gira alrededor de X. -->
@@ -520,4 +538,5 @@
   <axis xyz="-1.0 0.0 0.0"/>
   <dynamics damping="0.12" friction="0.03"/>
+  <xacro:arm_limit/>
 </joint>
 <!-- Brazo 3 (codo): gira alrededor de X. -->
@@ -528,4 +547,5 @@
   <axis xyz="1.0 0.0 0.0"/>
   <dynamics damping="0.12" friction="0.03"/>
+  <xacro:arm_limit/>
 </joint>
 <!-- Brazo 4 (muñeca): gira alrededor de X. -->
@@ -536,4 +556,5 @@
   <axis xyz="-1.0 0.0 0.0"/>
   <dynamics damping="0.06" friction="0.02"/>
+  <xacro:arm_limit/>
 </joint>
 <!-- Brazo 5 (muñeca): gira alrededor de Z. -->
@@ -544,4 +565,5 @@
   <axis xyz="0.0 0.0 1.0"/>
   <dynamics damping="0.05" friction="0.02"/>
+  <xacro:arm_limit/>
 </joint>
 <!-- Brazo 6 (muñeca): gira alrededor de X. -->
@@ -552,4 +574,5 @@
   <axis xyz="-1.0 0.0 0.0"/>
   <dynamics damping="0.05" friction="0.02"/>
+  <xacro:arm_limit/>
 </joint>
 <!-- Dedo derecho: se desliza en Y entre -7 mm y +16 mm. -->
@@ -569,4 +592,14 @@
   <xacro:unless value="${lock_arm}"><mimic joint="right_finger_joint" multiplier="-1.0" offset="0.0"/></xacro:unless>
   <limit upper="0.007" lower="-0.016" effort="30" velocity="0.05"/>
+</joint>
+<!-- Punto de agarre (TCP): centro entre las caras internas de los dedos, medido en sus mallas.
+     La pinza apunta hacia -X de link_6_1. Las caras internas van de x = -0.083 a -0.121 m
+     (la punta de los dedos está en -0.1224) y son simétricas en Y y Z. El TCP queda a la mitad.
+     Es el frame que mueve la cinemática inversa (andesrobot_arm). -->
+<link name="gripper_tcp"/>
+<joint name="gripper_tcp_joint" type="fixed">
+  <origin xyz="-0.102 0.0 0.0" rpy="0 0 0"/>
+  <parent link="link_6_1"/>
+  <child link="gripper_tcp"/>
 </joint>
 <!-- Elevador: el carro sube/baja en Z por la columna, de -0.4 m a +0.6 m. -->
@@ -682,3 +715,7 @@
   <xacro:include filename="$(find andesrobot_description)/urdf/andesrobot.ros2_control.xacro" />
 </xacro:if>
+<!-- Brazo en simulación: ros2_control con Gazebo (solo con arm_control:=true). -->
+<xacro:if value="${arm_control and not lock_arm}">
+  <xacro:include filename="$(find andesrobot_description)/urdf/andesrobot.arm_control.xacro" />
+</xacro:if>
 </robot>

Commit message: Brazo: masas reales (motores y pinza en ABS) y cámara Orbbec Gemini Plus sobre la pinza
Masas (andesrobot.urdf.xacro):
- La pinza EBG-20 es de ABS pero el CAD le asignó acero: masa e inercia de link_6_1 y los
  dedos escaladas con gripper_mass_scale (1.07 -> 0.14 kg) + servo de 55 g.
- Motores del EB300 como links fijos motor_joint_1..6 en el eslabón anterior a cada
  articulación (NEMA23 82 mm en joint_1 y 2, NEMA23 76 mm en joint_3, NEMA17 60 mm en
  joint_4 a 6). Brazo: 4.42 -> 8.05 kg. Reductores EBA en 0 hasta tener sus STL.

Cámara (gripper_camera:=true, activada en arm_sim con el argumento camara):
- andesrobot.gripper_camera.xacro: malla del modelo propio (orbbec_gemini_plus.stl), soporte
  con bisagra inclinado 20°, frames de cada lente y sensores de Gazebo de color, profundidad
  (+ nube) e infrarrojo, con los nombres de topic del driver real OrbbecSDK_ROS2.
- capturar_camara: guarda una imagen de cada canal en ros2_ws/capturas/ (fuera de git).
- worlds/mesa_prueba.sdf: mesa con tres objetos frente a Milo (argumento mesa).
- arm.rviz: paneles de color, profundidad e infrarrojo y la nube de puntos.
- Documentación en BRAZO.md, ROBOT.md, README.md y CLAUDE.md.

Co-Authored-By: Claude Opus 5.5 <noreply@anthropic.com>

File: ros2_ws/src/andesrobot_description/urdf/andesrobot.urdf.xacro (robot description, xacro)
@@ -56,4 +56,14 @@
 <xacro:arg name="sim_lidar" default="true"/>
 <xacro:arg name="sim_imu" default="true"/>
+<!-- MATERIAL DE LA PINZA (gripper EBG-20 de Toolbox Robotics)
+     Las masas de este archivo vienen del CAD de Fusion: masa = volumen de la pieza x densidad del
+     material que tenía asignado. Casi todo quedó en ABS macizo (1.06 g/cm3), pero la pinza
+     (link_6_1 y los dos dedos) quedó en acero (7.85 g/cm3, el material por defecto de Fusion):
+     pesaba 1.07 kg. La pinza real es de ABS impreso, así que su masa e inercia se multiplican por
+     1.06 / 7.85 (misma forma, otro material: la inercia escala igual que la masa).
+     Ver andesrobot_arm/docs/hardware/README.md. -->
+<xacro:property name="gripper_cad_density" value="7.85"/>  <!-- [g/cm3] acero, lo que usó el CAD -->
+<xacro:property name="gripper_density" value="1.06"/>      <!-- [g/cm3] ABS, el material real -->
+<xacro:property name="gripper_mass_scale" value="${gripper_density / gripper_cad_density}"/>
 <!--
   Convención REP-103 / REP-105 (estándar de ROS):
@@ -240,10 +250,11 @@
   </xacro:unless>
 </link>
-<!-- Brazo, eslabón 6: muñeca final, donde va la pinza. -->
+<!-- Brazo, eslabón 6: muñeca final, donde va la pinza. La malla es el cuerpo de la pinza EBG-20;
+     masa e inercia del CAD (acero) escaladas a ABS con gripper_mass_scale. -->
 <link name="link_6_1">
   <inertial>
     <origin xyz="-0.04672721914174861 0.0010341455962512703 -4.467579352440687e-05" rpy="0 0 0"/>
-    <mass value="0.7388320393848112"/>
-    <inertia ixx="0.000723" iyy="0.000493" izz="0.000757" ixy="5e-06" iyz="-1e-06" ixz="-1e-06"/>
+    <mass value="${0.7388320393848112 * gripper_mass_scale}"/>
+    <inertia ixx="${0.000723 * gripper_mass_scale}" iyy="${0.000493 * gripper_mass_scale}" izz="${0.000757 * gripper_mass_scale}" ixy="${5e-06 * gripper_mass_scale}" iyz="${-1e-06 * gripper_mass_scale}" ixz="${-1e-06 * gripper_mass_scale}"/>
   </inertial>
   <visual>
@@ -267,6 +278,6 @@
   <inertial>
     <origin xyz="-0.0246083952902236 0.013356716518430598 -0.007375101628988023" rpy="0 0 0"/>
-    <mass value="0.16542337365750662"/>
-    <inertia ixx="4.2e-05" iyy="6.6e-05" izz="8.3e-05" ixy="1.6e-05" iyz="9e-06" ixz="-1.6e-05"/>
+    <mass value="${0.16542337365750662 * gripper_mass_scale}"/>
+    <inertia ixx="${4.2e-05 * gripper_mass_scale}" iyy="${6.6e-05 * gripper_mass_scale}" izz="${8.3e-05 * gripper_mass_scale}" ixy="${1.6e-05 * gripper_mass_scale}" iyz="${9e-06 * gripper_mass_scale}" ixz="${-1.6e-05 * gripper_mass_scale}"/>
   </inertial>
   <visual>
@@ -290,6 +301,6 @@
   <inertial>
     <origin xyz="-0.024608395290223434 -0.013356716294173003 0.007375804549700549" rpy="0 0 0"/>
-    <mass value="0.16542337365750778"/>
-    <inertia ixx="4.2e-05" iyy="6.6e-05" izz="8.3e-05" ixy="-1.6e-05" iyz="9e-06" ixz="1.6e-05"/>
+    <mass value="${0.16542337365750778 * gripper_mass_scale}"/>
+    <inertia ixx="${4.2e-05 * gripper_mass_scale}" iyy="${6.6e-05 * gripper_mass_scale}" izz="${8.3e-05 * gripper_mass_scale}" ixy="${-1.6e-05 * gripper_mass_scale}" iyz="${9e-06 * gripper_mass_scale}" ixz="${1.6e-05 * gripper_mass_scale}"/>
   </inertial>
   <visual>
@@ -519,4 +530,82 @@
   </xacro:unless>
 </xacro:macro>
+<!-- ================= MOTORES DEL BRAZO (EB300 de Toolbox Robotics) =================
+  El CAD solo tiene las piezas impresas: los motores paso a paso no estaban en las masas.
+  Qué motor va en cada articulación sale de la guía eléctrica del EB300 (págs. 22-27); la masa,
+  de los datasheets de andesrobot_arm/docs/hardware/ (README.md):
+    joint_1, joint_2  NEMA23 82 mm  (23HS32-4004S, 2.4 N·m)  ~1.10 kg (el datasheet no la trae:
+                                                              extrapolada del de 3.10" = 1.07 kg)
+    joint_3           NEMA23 76 mm  (1.85 N·m)               ~1.07 kg
+    joint_4, 5, 6     NEMA17 60 mm  (0.65 N·m)               ~0.41 kg
+  Faltan los reductores planetarios impresos EBA-17/EBA-23: quedan en 0 hasta tener sus STL.
+  Cada motor va montado en el eslabón ANTERIOR a la articulación que mueve (el motor del hombro
+  va en la carcasa de link_1_1 y mueve link_2_1), coaxial con su eje. Se agrega como un link
+  fijo con solo <inertial>: Gazebo funde los links fijos con su padre, así que la masa, el
+  centro de masa y la inercia del eslabón quedan bien sin tocar los valores del CAD.
+  Simplificación: el centro del motor se pone en el origen de su articulación (sobre el eje).
+  Correrlo a lo largo del eje no cambia el torque que hace el peso en las articulaciones
+  paralelas a ese eje. Cuerpo del motor = caja de lado x lado x largo, con el largo en el eje. -->
+<xacro:property name="nema23_side" value="0.057"/>   <!-- [m] cara del NEMA23 -->
+<xacro:property name="nema17_side" value="0.042"/>   <!-- [m] cara del NEMA17 -->
+<xacro:property name="nema23_82_mass" value="1.10"/>  <!-- [kg] ver arriba -->
+<xacro:property name="nema23_76_mass" value="1.07"/>
+<xacro:property name="nema17_60_mass" value="0.41"/>
+<!-- arm_motor: un motor como link fijo.
+     parent / xyz / rpy = el mismo padre y origin que la articulación que mueve.
+     axis = eje del motor en ese frame ('x' o 'z'; el signo no importa para la inercia). -->
+<xacro:macro name="arm_motor" params="name parent xyz rpy mass side length axis">
+  <link name="${name}">
+    <inertial>
+      <origin xyz="0 0 0" rpy="0 0 0"/>
+      <mass value="${mass}"/>
+      <!-- Caja: I = m/12 (a² + b²) con a, b las medidas perpendiculares a cada eje. -->
+      <xacro:if value="${axis == 'x'}">
+        <inertia ixx="${mass/12*(2*side**2)}" ixy="0" ixz="0"
+                 iyy="${mass/12*(side**2 + length**2)}" iyz="0"
+                 izz="${mass/12*(side**2 + length**2)}"/>
+      </xacro:if>
+      <xacro:if value="${axis == 'z'}">
+        <inertia ixx="${mass/12*(side**2 + length**2)}" ixy="0" ixz="0"
+                 iyy="${mass/12*(side**2 + length**2)}" iyz="0"
+                 izz="${mass/12*(2*side**2)}"/>
+      </xacro:if>
+    </inertial>
+  </link>
+  <joint name="${name}_joint" type="fixed">
+    <origin xyz="${xyz}" rpy="${rpy}"/>
+    <parent link="${parent}"/>
+    <child link="${name}"/>
+  </joint>
+</xacro:macro>
+<!-- Un motor por articulación (xyz/rpy copiados del origin de cada joint_k, más abajo). -->
+<xacro:arm_motor name="motor_joint_1" parent="arm_base_link_1" xyz="0.0 0.0 0.037" rpy="0 0 0"
+                 mass="${nema23_82_mass}" side="${nema23_side}" length="0.082" axis="z"/>
+<xacro:arm_motor name="motor_joint_2" parent="link_1_1" xyz="-0.065 0.0 0.056" rpy="0 0 0"
+                 mass="${nema23_82_mass}" side="${nema23_side}" length="0.082" axis="x"/>
+<xacro:arm_motor name="motor_joint_3" parent="link_2_1" xyz="-0.001077 0.0 0.350077" rpy="0 0 0"
+                 mass="${nema23_76_mass}" side="${nema23_side}" length="0.076" axis="x"/>
+<xacro:arm_motor name="motor_joint_4" parent="link_3_1" xyz="0.026 0.0 0.3235" rpy="0 0 0"
+                 mass="${nema17_60_mass}" side="${nema17_side}" length="0.060" axis="x"/>
+<xacro:arm_motor name="motor_joint_5" parent="link_4_1" xyz="-0.0495 0.0 0.04" rpy="0 0 0"
+                 mass="${nema17_60_mass}" side="${nema17_side}" length="0.060" axis="z"/>
+<xacro:arm_motor name="motor_joint_6" parent="link_5_1" xyz="-0.041 0.0 0.0495" rpy="0 0 0"
+                 mass="${nema17_60_mass}" side="${nema17_side}" length="0.060" axis="x"/>
+<!-- Servo de la pinza (MG996R o similar, ~55 g), dentro del cuerpo de la pinza: en el centro de
+     link_6_1 (su malla va de x = -0.0725 a 0). Caja de 40 x 20 x 43 mm. -->
+<xacro:property name="gripper_servo_mass" value="0.055"/>
+<link name="gripper_servo_link">
+  <inertial>
+    <origin xyz="0 0 0" rpy="0 0 0"/>
+    <mass value="${gripper_servo_mass}"/>
+    <inertia ixx="${gripper_servo_mass/12*(0.020**2 + 0.043**2)}" ixy="0" ixz="0"
+             iyy="${gripper_servo_mass/12*(0.040**2 + 0.043**2)}" iyz="0"
+             izz="${gripper_servo_mass/12*(0.040**2 + 0.020**2)}"/>
+  </inertial>
+</link>
+<joint name="gripper_servo_joint" type="fixed">
+  <origin xyz="-0.036 0.0 0.0" rpy="0 0 0"/>
+  <parent link="link_6_1"/>
+  <child link="gripper_servo_link"/>
+</joint>
 <!-- Brazo 1: gira la base del brazo alrededor de Z (vertical). -->
 <joint name="joint_1" type="${arm_joint_type}">
@@ -719,3 +808,10 @@
   <xacro:include filename="$(find andesrobot_description)/urdf/andesrobot.arm_control.xacro" />
 </xacro:if>
+<!-- Cámara Orbbec Gemini Plus sobre la pinza (solo con gripper_camera:=true): cuerpo, soporte,
+     frames de cada lente y sus sensores en Gazebo (color, profundidad + nube, infrarrojo).
+     Por defecto no, así la simulación de mapeo no cambia. La activa andesrobot_arm/arm_sim.launch.py. -->
+<xacro:arg name="gripper_camera" default="false"/>
+<xacro:if value="$(arg gripper_camera)">
+  <xacro:include filename="$(find andesrobot_description)/urdf/andesrobot.gripper_camera.xacro" />
+</xacro:if>
 </robot>

Commit message: P04: topes por articulación en el xacro y hoja de medición del brazo real
Cada articulación tiene sus topes (joint_N_lower/upper, hoy ±π; el URDF
procesado queda idéntico). Hoja docs/medicion_brazo.md y script
comparar_medidas.py (con medidas.py, 4 pruebas) que compara lo medido con el
URDF y el DH del EB300 y escribe las líneas del xacro. PENDIENTES.md P04 con
lo hecho y lo que falta medir con el brazo armado.

Co-Authored-By: Claude Sonnet 5.5 <noreply@anthropic.com>
Claude-Session: https://claude.ai/code/session_01BmsU3Zui3kwJ8MywW7YE9T

File: ros2_ws/src/andesrobot_description/urdf/andesrobot.urdf.xacro (robot description, xacro)
@@ -520,13 +520,29 @@
      o sea sin restringir el rango), 20 N·m y 1 rad/s. Sirven para simular y para la cinemática
      inversa, pero NO son los topes reales: antes de mover el brazo real (o usar MoveIt), medir los
-     topes físicos y los motores y cambiar estas 4 propiedades. Con lock_arm:=true son "fixed". -->
+     topes físicos y los motores y cambiar estas propiedades. Con lock_arm:=true son "fixed".
+     Cada articulación tiene sus propios topes (joint_N_lower / joint_N_upper, en radianes, medidos
+     desde la pose cero del URDF y con el sentido positivo del eje de esa articulación). Mientras no
+     se midan, todos valen arm_lower / arm_upper (±π). Para poner un tope real basta cambiar el
+     número de la articulación que se midió; hoja de medición: docs/medicion_brazo.md. -->
 <xacro:property name="arm_lower" value="${-pi}"/>
 <xacro:property name="arm_upper" value="${pi}"/>
 <xacro:property name="arm_effort" value="20.0"/>
 <xacro:property name="arm_velocity" value="1.0"/>
+<xacro:property name="joint_1_lower" value="${arm_lower}"/>   <!-- [rad] provisorio -->
+<xacro:property name="joint_1_upper" value="${arm_upper}"/>
+<xacro:property name="joint_2_lower" value="${arm_lower}"/>
+<xacro:property name="joint_2_upper" value="${arm_upper}"/>
+<xacro:property name="joint_3_lower" value="${arm_lower}"/>
+<xacro:property name="joint_3_upper" value="${arm_upper}"/>
+<xacro:property name="joint_4_lower" value="${arm_lower}"/>
+<xacro:property name="joint_4_upper" value="${arm_upper}"/>
+<xacro:property name="joint_5_lower" value="${arm_lower}"/>
+<xacro:property name="joint_5_upper" value="${arm_upper}"/>
+<xacro:property name="joint_6_lower" value="${arm_lower}"/>
+<xacro:property name="joint_6_upper" value="${arm_upper}"/>
 <!-- Límite de cada articulación del brazo (las "fixed" no llevan límite). -->
-<xacro:macro name="arm_limit">
+<xacro:macro name="arm_limit" params="lower upper">
   <xacro:unless value="${lock_arm}">
-    <limit lower="${arm_lower}" upper="${arm_upper}" effort="${arm_effort}" velocity="${arm_velocity}"/>
+    <limit lower="${lower}" upper="${upper}" effort="${arm_effort}" velocity="${arm_velocity}"/>
   </xacro:unless>
 </xacro:macro>
@@ -619,5 +635,5 @@
   <!-- Amortiguación y roce de la articulación (solo para la simulación). -->
   <dynamics damping="0.08" friction="0.02"/>
-  <xacro:arm_limit/>
+  <xacro:arm_limit lower="${joint_1_lower}" upper="${joint_1_upper}"/>
 </joint>
 <!-- Brazo 2 (hombro): gira alrededor de X. -->
@@ -628,5 +644,5 @@
   <axis xyz="-1.0 0.0 0.0"/>
   <dynamics damping="0.12" friction="0.03"/>
-  <xacro:arm_limit/>
+  <xacro:arm_limit lower="${joint_2_lower}" upper="${joint_2_upper}"/>
 </joint>
 <!-- Brazo 3 (codo): gira alrededor de X. -->
@@ -637,5 +653,5 @@
   <axis xyz="1.0 0.0 0.0"/>
   <dynamics damping="0.12" friction="0.03"/>
-  <xacro:arm_limit/>
+  <xacro:arm_limit lower="${joint_3_lower}" upper="${joint_3_upper}"/>
 </joint>
 <!-- Brazo 4 (muñeca): gira alrededor de X. -->
@@ -646,5 +662,5 @@
   <axis xyz="-1.0 0.0 0.0"/>
   <dynamics damping="0.06" friction="0.02"/>
-  <xacro:arm_limit/>
+  <xacro:arm_limit lower="${joint_4_lower}" upper="${joint_4_upper}"/>
 </joint>
 <!-- Brazo 5 (muñeca): gira alrededor de Z. -->
@@ -655,5 +671,5 @@
   <axis xyz="0.0 0.0 1.0"/>
   <dynamics damping="0.05" friction="0.02"/>
-  <xacro:arm_limit/>
+  <xacro:arm_limit lower="${joint_5_lower}" upper="${joint_5_upper}"/>
 </joint>
 <!-- Brazo 6 (muñeca): gira alrededor de X. -->
@@ -664,5 +680,5 @@
   <axis xyz="-1.0 0.0 0.0"/>
   <dynamics damping="0.05" friction="0.02"/>
-  <xacro:arm_limit/>
+  <xacro:arm_limit lower="${joint_6_lower}" upper="${joint_6_upper}"/>
 </joint>
 <!-- Dedo derecho: se desliza en Y entre -7 mm y +16 mm. -->
